Commit message: Second and third joints.

File: urdf/thor_robot.urdf (robot description, URDF)
Before this commit: robot thor, 2 links, 1 joints
Links:
- added link art2; visual mesh filename=package://thor_arm_description/meshes/art2.stl scale=0.001 0.001 0.001
- added link art3; visual mesh filename=package://thor_arm_description/meshes/art3.stl scale=0.001 0.001 0.001
- link art1: mass 1 -> None
Joints:
- added joint art2_pitch: type revolute, parent art1, child art2, origin xyz=0 -0.0318752 0.0974304 rpy=1.5707963267948966 -1.5707963267948966 0, axis 0 0 1, limit lower=-1.5707963267948966 upper=1.5707963267948966 effort=4 velocity=1
- added joint art3_pitch: type revolute, parent art2, child art3, origin xyz=0.160 0 0 rpy=0 0 0, axis 0 0 1, limit lower=-1.5707963267948966 upper=1.5707963267948966 effort=4 velocity=1
- joint art1_yaw: axis (none) -> 0 0 1; origin xyz=0 0 0.104 rpy=0 -1.5707963267948966 0 -> xyz=0 0 0.104 rpy=0 0 0

Commit message: Fourth joint.

File: urdf/thor_robot.urdf (robot description, URDF)
Before this commit: robot thor, 4 links, 3 joints
Links:
- added link art4; visual mesh filename=package://thor_arm_description/meshes/art4.stl scale=0.001 0.001 0.001
Joints:
- added joint art4_roll: type revolute, parent art3, child art4, origin xyz=0.0885 0 -0.035 rpy=0 1.5707963267948966 0, axis 0 0 1, limit lower=-1.5707963267948966 upper=1.5707963267948966 effort=4 velocity=1

Commit message: Fifth joint.

File: urdf/thor_robot.urdf (robot description, URDF)
Before this commit: robot thor, 5 links, 4 joints
Links:
- added link art5; visual mesh filename=package://thor_arm_description/meshes/art5.stl scale=0.001 0.001 0.001
Joints:
- added joint art5_pitch: type revolute, parent art4, child art5, origin xyz=0 0 0.1 rpy=0 -1.5707963267948966 0, axis 0 0 1, limit lower=-1.5707963267948966 upper=1.5707963267948966 effort=4 velocity=1

Commit message: Sixth joint.

File: urdf/thor_robot.urdf (robot description, URDF)
Before this commit: robot thor, 6 links, 5 joints
Links:
- added link art6; visual mesh filename=package://thor_arm_description/meshes/art6.stl scale=0.001 0.001 0.001
Joints:
- added joint art6_roll: type revolute, parent art5, child art6, origin xyz=0 0 0 rpy=0 1.5707963267948966 0, axis 0 0 1, limit lower=-1.5707963267948966 upper=1.5707963267948966 effort=4 velocity=1

Commit message: Expanded joint limits. Changed to a more neutral color.

File: urdf/thor_robot.urdf (robot description, URDF)
Before this commit: robot thor, 7 links, 6 joints
Joints:
- joint art4_roll: limit lower=-1.5707963267948966 upper=1.5707963267948966 effort=4 velocity=1 -> lower=-3.1415 upper=3.1415 effort=4 velocity=1
- joint art5_pitch: limit lower=-1.5707963267948966 upper=1.5707963267948966 effort=4 velocity=1 -> lower=-1.5 upper=1.5 effort=4 velocity=1
- joint art6_roll: limit lower=-1.5707963267948966 upper=1.5707963267948966 effort=4 velocity=1 -> lower=-3.1415 upper=3.1415 effort=4 velocity=1
